File: hardware/pcb/wled_0.0/wled_0.0.kicad_pcb (KiCad board)
At the start: 2 copper layers, 26 x 40.5 mm, 13 parts, among them J1 Conn_01x02_Female, J2 Conn_01x03_Female, Q1 BSS138, U1 AMS1117-3.3, U2 ESP-12

Commit message: увеличил размер переходных отверстий с 0.8 до 0.9
Other:
- net class Default: via_dia 0.8 -> 0.9

Commit message: поменял разъемы с вертикальных на горизонтальные
+ перенес на другую сторону(как было запаяно на тестовых платах)
Parts:
- J1: footprint Connector_PinHeader_2.54mm:PinHeader_1x02_P2.54mm_Vertical -> Connector_PinHeader_2.54mm:PinHeader_1x02_P2.54mm_Horizontal; moved to B.Cu
- J2: footprint Connector_PinHeader_2.54mm:PinHeader_1x03_P2.54mm_Vertical -> Connector_PinHeader_2.54mm:PinHeader_1x03_P2.54mm_Horizontal; moved to B.Cu
- turned J1 to 270 degrees
- turned J2 to 90 degrees
